File: AS5048Encoder/AS5048 Encoder/AS5048 Encoder.sch (EAGLE design)
At the start: 4 parts

Commit message: pre route
Parts:
- added X1: SI-50170, con-stewart:SI-50170
Connections:
- net GND: now also X1.TD-
- net PWM: now also X1.TCT
- net VCC: now also X1.TD+
Changed lines of the file:
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@@
 <?xml version="1.0" encoding="utf-8"?>
 <!DOCTYPE eagle SYSTEM "eagle.dtd">
-<eagle version="6.6.0">
+<eagle version="7.6.0">
 <drawing>
 <settings>
@@
 <part name="JP1" library="SparkFun-Connectors" deviceset="M03" device="LOCK"/>
 <part name="U$1" library="austriamicrosystems" deviceset="AS5048" device=""/>
+<part name="X1" library="con-stewart" deviceset="SI-50170" device=""/>
 </parts>
 <sheets>
@@
 <instance part="JP1" gate="G$1" x="63.5" y="58.42" rot="R270"/>
 <instance part="U$1" gate="G$1" x="66.04" y="25.4"/>
+<instance part="X1" gate="G$1" x="66.04" y="-7.62"/>
 </instances>
 <busses>
@@
 <label x="60.96" y="40.64" size="1.778" layer="95" rot="R90"/>
 </segment>
+<segment>
+<pinref part="X1" gate="G$1" pin="TD-"/>
+<wire x1="55.88" y1="2.54" x2="53.34" y2="2.54" width="0.1524" layer="91"/>
+<label x="48.26" y="2.54" size="1.778" layer="95"/>
+</segment>
 </net>
 <net name="VCC" class="0">
@@
 <label x="63.5" y="40.64" size="1.778" layer="95" rot="R90"/>
 </segment>
+<segment>
+<pinref part="X1" gate="G$1" pin="TD+"/>
+<wire x1="55.88" y1="7.62" x2="53.34" y2="7.62" width="0.1524" layer="91"/>
+<label x="48.26" y="7.62" size="1.778" layer="95"/>
+</segment>
 </net>
 <net name="3V3" class="0">
@@
 <label x="66.04" y="40.64" size="1.778" layer="95" rot="R90"/>
 </segment>
-</net>
+<segment>
+<pinref part="X1" gate="G$1" pin="TCT"/>
+<wire x1="55.88" y1="5.08" x2="53.34" y2="5.08" width="0.1524" layer="91"/>
+<label x="48.26" y="5.08" size="1.778" layer="95"/>
+</segment>
+</net>
