File: AS5048Encoder/AS5048 Encoder/AS5048 Encoder.brd (EAGLE design)
At the start: 50 x 50 mm, 6 parts

Commit message: real end of day
Parts:
- moved U$1 8.78 mm to (24.0, 32.1)
Other:
- board size 50 x 50 mm -> 43.1 x 39.9 mm
Changed lines of the file:
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@@
 <setting verticaltext="up"/>
 </settings>
-<grid distance="0.01778" unitdist="mm" unit="mm" style="lines" multiple="1" display="yes" altdistance="0.1" altunitdist="mm" altunit="mm"/>
+<grid distance="0.1" unitdist="mm" unit="mm" style="lines" multiple="1" display="yes" altdistance="0.1" altunitdist="mm" altunit="mm"/>
 <layers>
 <layer number="1" name="Top" color="4" fill="1" visible="yes" active="yes"/>
@@
 <board>
 <plain>
-<wire x1="0" y1="0" x2="0" y2="50" width="0" layer="20"/>
-<wire x1="0" y1="50" x2="50" y2="50" width="0" layer="20"/>
-<wire x1="50" y1="0" x2="0" y2="0" width="0" layer="20"/>
+<wire x1="2.99820625" y1="12.4210125" x2="15.648090625" y2="39.402509375" width="0" layer="20"/>
+<wire x1="15.648090625" y1="39.402509375" x2="20.2365375" y2="42.296328125" width="0" layer="20" curve="-65.285076"/>
+<wire x1="20.2365375" y1="42.296328125" x2="29.93720625" y2="42.2279375" width="0" layer="20"/>
+<wire x1="29.93720625" y1="42.2279375" x2="35.228496875" y2="38.466415625" width="0" layer="20" curve="-70.008043"/>
+<wire x1="35.228496875" y1="38.466415625" x2="45.124703125" y2="10.6543" width="0" layer="20"/>
+<wire x1="45.124703125" y1="10.6543" x2="39.230084375" y2="2.3483375" width="0" layer="20" curve="-109.89904"/>
+<wire x1="39.230084375" y1="2.3483375" x2="9.367134375" y2="2.511121875" width="0" layer="20"/>
+<wire x1="9.367134375" y1="2.511121875" x2="2.99820625" y2="12.4210125" width="0" layer="20" curve="-115.693887"/>
 <rectangle x1="22.85508125" y1="33.382346875" x2="23.7796375" y2="33.400121875" layer="200" rot="R270"/>
 <rectangle x1="22.72173125" y1="33.373453125" x2="23.94855" y2="33.391234375" layer="200" rot="R270"/>
@@
 <attribute name="VALUE" x="30.18431875" y="12.93114375" size="1.27" layer="27"/>
 </element>
-<element name="U$1" library="austriamicrosystems" package="TSOP14" value="AS5048" x="23.186640625" y="40.828478125" smashed="yes" rot="R270">
-<attribute name="VALUE" x="20.114978125" y="43.801615625" size="1.27" layer="27"/>
+<element name="U$1" library="austriamicrosystems" package="TSOP14" value="AS5048" x="24.04308125" y="32.08571875" smashed="yes" rot="R270">
+<attribute name="VALUE" x="20.97141875" y="35.05885625" size="1.27" layer="27"/>
 </element>
 <element name="U$2" library="SparkFun-Electromechanical" package="STAND-OFF-TIGHT" value="" x="38" y="10"/>
@@
 <contactref element="JP1" pad="1"/>
 <contactref element="U$1" pad="13"/>
-<wire x1="19.3598625" y1="13.544021875" x2="26.252059375" y2="42.174159375" width="0" layer="19" extent="1-1"/>
+<wire x1="19.3598625" y1="13.544021875" x2="27.1085" y2="33.4314" width="0" layer="19" extent="1-1"/>
 <wire x1="14.77528125" y1="13.97408125" x2="19.3598625" y2="13.544021875" width="0" layer="19" extent="1-1"/>
 <wire x1="31.45431875" y1="16.23314375" x2="19.3598625" y2="13.544021875" width="0" layer="19" extent="1-1"/>
@@
 <contactref element="JP1" pad="2"/>
 <contactref element="U$1" pad="11"/>
-<wire x1="19.3598625" y1="16.844021875" x2="26.252059375" y2="40.874159375" width="0" layer="19" extent="1-1"/>
+<wire x1="19.3598625" y1="16.844021875" x2="27.1085" y2="32.1314" width="0" layer="19" extent="1-1"/>
 <wire x1="33.99431875" y1="15.97914375" x2="19.3598625" y2="16.844021875" width="0" layer="19" extent="1-1"/>
 </signal>
@@
 <contactref element="C4" pad="A"/>
 <contactref element="U$1" pad="12"/>
-<wire x1="14.77528125" y1="17.27408125" x2="26.252059375" y2="41.524159375" width="0" layer="19" extent="1-1"/>
+<wire x1="14.77528125" y1="17.27408125" x2="27.1085" y2="32.7814" width="0" layer="19" extent="1-1"/>
 </signal>
 <signal name="PWM">
 <contactref element="U$1" pad="14"/>
 <contactref element="JP1" pad="3"/>
-<wire x1="36.53431875" y1="16.23314375" x2="26.252059375" y2="42.828478125" width="0" layer="19" extent="1-1"/>
+<wire x1="36.53431875" y1="16.23314375" x2="27.1085" y2="34.08571875" width="0" layer="19" extent="1-1"/>
 </signal>
 </signals>

Commit message: pre route
Parts:
- removed U$2, U$3: (no value), SparkFun-Electromechanical:STAND-OFF-TIGHT
- added X1: SI-50170, con-stewart:SI-50170
- moved C3 22.3 mm to (27.3, 36.1)
- moved C4 22.1 mm to (23.4, 36.0)
- moved U$1 12.0 mm to (25.0, 44.0)
- moved JP1 6.10 mm to (32.6, 22.1)
Connections:
- net GND: now also X1.3
- net PWM: now also X1.2
- net VCC: now also X1.1
Other:
- board size 43.1 x 39.9 mm -> 50 x 50 mm

Commit message: before rounding corners
Parts:
- moved C4 1.30 mm to (24.6, 36.5)
- moved C3 0.57 mm to (27.7, 36.5)
Routing:
- net PWM: track 0.00 -> 56.9 mm
- net GND: track 0.00 -> 50.6 mm
- net VCC: track 0.00 -> 46.9 mm
- net 3V3: track 0.00 -> 9.12 mm
Changed lines of the file:
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@@
 <setting verticaltext="up"/>
 </settings>
-<grid distance="0.1" unitdist="mm" unit="mm" style="lines" multiple="1" display="yes" altdistance="0.1" altunitdist="mm" altunit="mm"/>
+<grid distance="3.93700787" unitdist="mil" unit="mil" style="lines" multiple="1" display="yes" altdistance="0.1" altunitdist="mm" altunit="mm"/>
 <layers>
 <layer number="1" name="Top" color="4" fill="1" visible="yes" active="yes"/>
@@
 </autorouter>
 <elements>
-<element name="C3" library="SparkFun-Passives" package="EIA3216-KIT" value="100nF" x="27.2598625" y="36.094021875" smashed="yes" rot="R90">
-<attribute name="VALUE" x="32.542659375" y="39.35181875" size="1.27" layer="27" rot="R180"/>
+<element name="C3" library="SparkFun-Passives" package="EIA3216-KIT" value="100nF" x="27.6598625" y="36.494021875" smashed="yes" rot="R90">
+<attribute name="VALUE" x="27.14818125" y="32.342659375" size="1.27" layer="27" rot="R270"/>
 </element>
-<element name="C4" library="SparkFun-Passives" package="EIA3216-KIT" value="10uF" x="23.37528125" y="36.02408125" smashed="yes" rot="R90">
-<attribute name="VALUE" x="19.262078125" y="39.168440625" size="1.27" layer="27" rot="R180"/>
+<element name="C4" library="SparkFun-Passives" package="EIA3216-KIT" value="10uF" x="24.57528125" y="36.52408125" smashed="yes" rot="R90">
+<attribute name="VALUE" x="24.231559375" y="32.662078125" size="1.27" layer="27" rot="R270"/>
 </element>
 <element name="JP1" library="SparkFun-Connectors" package="1X03_LOCK" value="" x="32.55431875" y="22.10614375" smashed="yes">
@@
 <contactref element="U$1" pad="13"/>
 <contactref element="X1" pad="3"/>
-<wire x1="27.2598625" y1="34.444021875" x2="28.06541875" y2="45.34568125" width="0" layer="19" extent="1-1"/>
-<wire x1="23.37528125" y1="34.37408125" x2="27.2598625" y2="34.444021875" width="0" layer="19" extent="1-1"/>
-<wire x1="32.55431875" y1="22.23314375" x2="27.2598625" y2="34.444021875" width="0" layer="19" extent="1-1"/>
-<wire x1="23.095" y1="12.242" x2="23.37528125" y2="34.37408125" width="0" layer="19" extent="1-1"/>
+<wire x1="28.06541875" y1="45.34568125" x2="24.94568125" y2="45.34568125" width="0.4064" layer="1"/>
+<wire x1="24.94568125" y1="45.34568125" x2="23.8" y2="44.2" width="0.4064" layer="1"/>
+<wire x1="23.8" y1="44.2" x2="23.8" y2="41.6" width="0.4064" layer="1"/>
+<wire x1="23.8" y1="41.6" x2="21.6" y2="39.4" width="0.4064" layer="1"/>
+<wire x1="21.6" y1="39.4" x2="21.6" y2="35.4" width="0.4064" layer="1"/>
+<wire x1="21.6" y1="35.4" x2="22.5" y2="34.5" width="0.4064" layer="1"/>
+<wire x1="22.5" y1="34.5" x2="24.2012" y2="34.5" width="0.4064" layer="1"/>
+<wire x1="24.2012" y1="34.5" x2="24.57528125" y2="34.87408125" width="0.4064" layer="1"/>
+<wire x1="24.57528125" y1="34.87408125" x2="27.629803125" y2="34.87408125" width="0.4064" layer="1"/>
+<wire x1="27.629803125" y1="34.87408125" x2="27.6598625" y2="34.844021875" width="0.4064" layer="1"/>
+<wire x1="32.55431875" y1="22.23314375" x2="32.55431875" y2="29.949565625" width="0.4064" layer="1"/>
+<wire x1="32.55431875" y1="29.949565625" x2="27.6598625" y2="34.844021875" width="0.4064" layer="1"/>
+<wire x1="32.55431875" y1="22.23314375" x2="30.83314375" y2="22.23314375" width="0.4064" layer="1"/>
+<wire x1="30.83314375" y1="22.23314375" x2="23.2" y2="14.6" width="0.4064" layer="1"/>
+<wire x1="23.2" y1="14.6" x2="23.2" y2="12.347" width="0.4064" layer="1"/>
+<wire x1="23.2" y1="12.347" x2="23.095" y2="12.242" width="0.4064" layer="1"/>
 </signal>
 <signal name="VCC">
@@
 <contactref element="U$1" pad="11"/>
 <contactref element="X1" pad="1"/>
-<wire x1="27.2598625" y1="37.744021875" x2="28.06541875" y2="44.04568125" width="0" layer="19" extent="1-1"/>
-<wire x1="35.09431875" y1="21.97914375" x2="27.2598625" y2="37.744021875" width="0" layer="19" extent="1-1"/>
-<wire x1="20.555" y1="12.242" x2="27.2598625" y2="37.744021875" width="0" layer="19" extent="1-1"/>
+<wire x1="27.6598625" y1="38.144021875" x2="30.4" y2="40.884159375" width="0.4064" layer="1"/>
+<wire x1="30.4" y1="40.884159375" x2="30.4" y2="43.2" width="0.4064" layer="1"/>
+<wire x1="30.4" y1="43.2" x2="29.55431875" y2="44.04568125" width="0.4064" layer="1"/>
+<wire x1="29.55431875" y1="44.04568125" x2="28.06541875" y2="44.04568125" width="0.4064" layer="1"/>
+<wire x1="35.09431875" y1="21.97914375" x2="35.09431875" y2="30.709565625" width="0.4064" layer="1"/>
+<wire x1="35.09431875" y1="30.709565625" x2="27.6598625" y2="38.144021875" width="0.4064" layer="1"/>
+<wire x1="20.555" y1="12.242" x2="20.555" y2="12.655" width="0.4064" layer="16"/>
+<wire x1="20.555" y1="12.655" x2="27.7" y2="19.8" width="0.4064" layer="16"/>
+<wire x1="27.7" y1="19.8" x2="32.915175" y2="19.8" width="0.4064" layer="16"/>
+<wire x1="32.915175" y1="19.8" x2="35.09431875" y2="21.97914375" width="0.4064" layer="16"/>
 </signal>
 <signal name="3V3">
 <contactref element="C4" pad="A"/>
 <contactref element="U$1" pad="12"/>
-<wire x1="23.37528125" y1="37.67408125" x2="28.06541875" y2="44.69568125" width="0" layer="19" extent="1-1"/>
+<wire x1="24.57528125" y1="38.17408125" x2="25.1" y2="38.6988" width="0.4064" layer="1"/>
+<wire x1="25.1" y1="38.6988" x2="25.1" y2="43.7" width="0.4064" layer="1"/>
+<wire x1="25.1" y1="43.7" x2="26.09568125" y2="44.69568125" width="0.4064" layer="1"/>
+<wire x1="26.09568125" y1="44.69568125" x2="28.06541875" y2="44.69568125" width="0.4064" layer="1"/>
 </signal>
 <signal name="PWM">
@@
 <contactref element="JP1" pad="3"/>
 <contactref element="X1" pad="2"/>
-<wire x1="37.63431875" y1="22.23314375" x2="28.06541875" y2="46" width="0" layer="19" extent="1-1"/>
-<wire x1="21.825" y1="9.702" x2="37.63431875" y2="22.23314375" width="0" layer="19" extent="1-1"/>
+<wire x1="37.63431875" y1="22.23314375" x2="37.63431875" y2="40.26568125" width="0.4064" layer="1"/>
+<wire x1="37.63431875" y1="40.26568125" x2="31.9" y2="46" width="0.4064" layer="1"/>
+<wire x1="31.9" y1="46" x2="28.06541875" y2="46" width="0.4064" layer="1"/>
+<wire x1="21.825" y1="9.702" x2="24.227" y2="7.3" width="0.4064" layer="1"/>
+<wire x1="24.227" y1="7.3" x2="29.4" y2="7.3" width="0.4064" layer="1"/>
+<wire x1="29.4" y1="7.3" x2="37.63431875" y2="15.53431875" width="0.4064" layer="1"/>
+<wire x1="37.63431875" y1="15.53431875" x2="37.63431875" y2="22.23314375" width="0.4064" layer="1"/>
 </signal>
 </signals>
